File: Hardware/Controllerv1/PrinterController/_saved_Power.sch (KiCad schematic (older format))
At the start: 2 parts

Commit message: Added pcb changes
Parts:
- removed J?: Screw_Terminal_01x04, symbol Screw_Terminal_01x04
- added J22, J24: Screw_Terminal_01x02, TerminalBlocks_WAGO:TerminalBlock_WAGO-804_RM7.5mm_2pol, symbol Screw_Terminal_01x02
- J23: renamed from J?; footprint (none) -> Connectors_Molex:Molex_KK-6410-03_03x2.54mm_Straight
Connections:
- net +VDC: now also J24.2 (Pin_2)
- net GNDPWR: now also J22.1 (Pin_1), J24.1 (Pin_1)
- new net VAA: J22.2 (Pin_2)
Changed lines of the file:
@@
 Comment4 ""
 $EndDescr
-$Comp
-L Screw_Terminal_01x04 J?
-U 1 1 5B2F4D3D
-P 1100 1300
-F 0 "J?" H 1100 1500 50  0000 C CNN
-F 1 "Screw_Terminal_01x04" H 1100 1000 50  0000 C CNN
-F 2 "" H 1100 1300 50  0001 C CNN
-F 3 "" H 1100 1300 50  0001 C CNN
-	1    1100 1300
-	-1   0    0    1
-$EndComp
-$Comp
-L +VDC #PWR?
-U 1 1 5B2F4DEF
-P 1650 850
-F 0 "#PWR?" H 1650 750 50  0001 C CNN
-F 1 "+VDC" H 1650 1100 50  0000 C CNN
-F 2 "" H 1650 850 50  0001 C CNN
-F 3 "" H 1650 850 50  0001 C CNN
-	1    1650 850
-	1    0    0    -1
-$EndComp
-Wire Wire Line
-	1650 850  1650 1200
 Wire Wire Line
 	1650 1100 1300 1100
-Wire Wire Line
-	1650 1200 1300 1200
-Connection ~ 1650 1100
 $Comp
-L GNDPWR #PWR?
+L GNDPWR #PWR52
 U 1 1 5B2F4E32
 P 1650 1450
-F 0 "#PWR?" H 1650 1250 50  0001 C CNN
+F 0 "#PWR52" H 1650 1250 50  0001 C CNN
 F 1 "GNDPWR" H 1650 1320 50  0000 C CNN
 F 2 "" H 1650 1400 50  0001 C CNN
@@
 $EndComp
 Wire Wire Line
-	1650 1450 1650 1300
-Wire Wire Line
-	1650 1300 1300 1300
-Wire Wire Line
 	1300 1400 1650 1400
-Connection ~ 1650 1400
 Text Notes 550  750  0    60   ~ 0
 +12-24V Input\n
@@
 Digital Voltage (3.3 and 5V)\n
 $Comp
-L Conn_01x03 J?
+L Conn_01x03 J23
 U 1 1 5B2F4EB7
 P 1100 2200
-F 0 "J?" H 1100 2400 50  0000 C CNN
+F 0 "J23" H 1100 2400 50  0000 C CNN
 F 1 "Conn_01x03" H 1100 2000 50  0000 C CNN
-F 2 "" H 1100 2200 50  0001 C CNN
+F 2 "Connectors_Molex:Molex_KK-6410-03_03x2.54mm_Straight" H 1100 2200 50  0001 C CNN
 F 3 "" H 1100 2200 50  0001 C CNN
 	1    1100 2200
@@
 $EndComp
 $Comp
-L +5V #PWR?
+L +5V #PWR49
 U 1 1 5B2F4EF4
 P 1550 2050
-F 0 "#PWR?" H 1550 1900 50  0001 C CNN
+F 0 "#PWR49" H 1550 1900 50  0001 C CNN
 F 1 "+5V" H 1550 2190 50  0000 C CNN
 F 2 "" H 1550 2050 50  0001 C CNN
@@
 $EndComp
 $Comp
-L +3V3 #PWR?
+L +3V3 #PWR53
 U 1 1 5B2F4F0C
 P 1750 2050
-F 0 "#PWR?" H 1750 1900 50  0001 C CNN
+F 0 "#PWR53" H 1750 1900 50  0001 C CNN
 F 1 "+3V3" H 1750 2190 50  0000 C CNN
 F 2 "" H 1750 2050 50  0001 C CNN
@@
 $EndComp
 $Comp
-L GND #PWR?
+L GND #PWR50
 U 1 1 5B2F4F24
 P 1550 2350
-F 0 "#PWR?" H 1550 2100 50  0001 C CNN
+F 0 "#PWR50" H 1550 2100 50  0001 C CNN
 F 1 "GND" H 1550 2200 50  0000 C CNN
 F 2 "" H 1550 2350 50  0001 C CNN
@@
 Wire Wire Line
 	1550 2100 1550 2050
+$Comp
+L Screw_Terminal_01x02 J22
+U 1 1 5B315F3F
+P 1100 1200
+F 0 "J22" H 1100 950 50  0000 C CNN
+F 1 "Screw_Terminal_01x02" H 1100 1000 50  0000 C CNN
+F 2 "TerminalBlocks_WAGO:TerminalBlock_WAGO-804_RM7.5mm_2pol" H 1100 1200 50  0001 C CNN
+F 3 "" H 1100 1200 50  0001 C CNN
+	1    1100 1200
+	-1   0    0    1
+$EndComp
+$Comp
+L Screw_Terminal_01x02 J24
+U 1 1 5B315F58
+P 1100 1400
+F 0 "J24" H 1100 1500 50  0000 C CNN
+F 1 "Screw_Terminal_01x02" H 1200 1600 50  0000 C CNN
+F 2 "TerminalBlocks_WAGO:TerminalBlock_WAGO-804_RM7.5mm_2pol" H 1100 1400 50  0001 C CNN
+F 3 "" H 1100 1400 50  0001 C CNN
+	1    1100 1400
+	-1   0    0    1
+$EndComp
+$Comp
+L VAA #PWR51
+U 1 1 5B316A86
+P 1650 1100
+F 0 "#PWR51" H 1650 950 50  0001 C CNN
+F 1 "VAA" H 1650 1250 50  0000 C CNN
+F 2 "" H 1650 1100 50  0001 C CNN
+F 3 "" H 1650 1100 50  0001 C CNN
+	1    1650 1100
+	1    0    0    -1
+$EndComp
+Wire Wire Line
+	1300 1300 1800 1300
+Wire Wire Line
+	1800 1300 1800 1100
+$Comp
+L +VDC #PWR54
+U 1 1 5B316AE9
+P 1800 1100
+F 0 "#PWR54" H 1800 1000 50  0001 C CNN
+F 1 "+VDC" H 1800 1350 50  0000 C CNN
+F 2 "" H 1800 1100 50  0001 C CNN
+F 3 "" H 1800 1100 50  0001 C CNN
+	1    1800 1100
+	1    0    0    -1
+$EndComp
+Wire Wire Line
+	1650 1200 1650 1450
+Wire Wire Line
+	1300 1200 1650 1200
+Connection ~ 1650 1400
 $EndSCHEMATC
