File: Hardware/Controllerv1/PrinterController/Motor.sch (KiCad schematic (older format))
At the start: 0 parts

Commit message: Added updates to PCB
Parts:
- added J10, J11, J9: Conn_02x03_Odd_Even, Pin_Headers:Pin_Header_Straight_2x03_Pitch1.27mm_SMD, symbol Conn_02x03_Odd_Even
- added J12, J13, J14, J15, J16, J17, J18, J19, J6, J7, J8: Conn_01x04, Socket_Strips:Socket_Strip_Straight_1x04_Pitch2.54mm, symbol Conn_01x04
- added J20, J21: Conn_02x03_Odd_Even, symbol Conn_02x03_Odd_Even
- added U12, U13, U14, U15, U16, U17: pololu_DRV8825, .pretty:DRV8825, symbol pololu_DRV8825
Connections:
- new net: J12.4 (Pin_4), U12.11 (A2)
- new net: J12.3 (Pin_3), U12.12 (A1)
- new net: J12.2 (Pin_2), U12.13 (B1)
- new net: J12.1 (Pin_1), U12.14 (B2)
- new net: J10.2 (Pin_2), U12.2 (M0)
- new net: J10.4 (Pin_4), U12.3 (M1)
- new net: J10.6 (Pin_6), U12.4 (M2)
- new net: J13.4 (Pin_4), U13.11 (A2)
- new net: J13.3 (Pin_3), U13.12 (A1)
- new net: J13.2 (Pin_2), U13.13 (B1)
- new net: J13.1 (Pin_1), U13.14 (B2)
- new net: J11.2 (Pin_2), U13.2 (M0)
- new net: J11.4 (Pin_4), U13.3 (M1)
- new net: J11.6 (Pin_6), U13.4 (M2)
- new net: J14.4 (Pin_4), U14.11 (A2)
- new net: J14.3 (Pin_3), U14.12 (A1)
- new net: J14.2 (Pin_2), U14.13 (B1)
- new net: J14.1 (Pin_1), U14.14 (B2)
- new net: J9.2 (Pin_2), U14.2 (M0), U15.2 (M0)
- new net: J9.4 (Pin_4), U14.3 (M1), U15.3 (M1)
- new net: J9.6 (Pin_6), U14.4 (M2), U15.4 (M2)
- new net: J15.4 (Pin_4), U15.11 (A2)
- new net: J15.3 (Pin_3), U15.12 (A1)
- new net: J15.2 (Pin_2), U15.13 (B1)
- new net: J15.1 (Pin_1), U15.14 (B2)
- new net: J16.4 (Pin_4), U16.11 (A2)
- new net: J16.3 (Pin_3), U16.12 (A1)
- new net: J16.2 (Pin_2), U16.13 (B1)
- new net: J16.1 (Pin_1), U16.14 (B2)
- new net: J20.2 (Pin_2), U16.2 (M0)
- new net: J20.4 (Pin_4), U16.3 (M1)
- new net: J20.6 (Pin_6), U16.4 (M2)
- new net: J17.4 (Pin_4), U17.11 (A2)
- new net: J17.3 (Pin_3), U17.12 (A1)
- new net: J17.2 (Pin_2), U17.13 (B1)
- new net: J17.1 (Pin_1), U17.14 (B2)
- new net: J21.2 (Pin_2), U17.2 (M0)
- new net: J21.4 (Pin_4), U17.3 (M1)
- new net: J21.6 (Pin_6), U17.4 (M2)
- new net +3V3: J10.1 (Pin_1), J10.3 (Pin_3), J10.5 (Pin_5), J11.1 (Pin_1), J11.3 (Pin_3), J11.5 (Pin_5), J20.1 (Pin_1), J20.3 (Pin_3), J20.5 (Pin_5), J21.1 (Pin_1), J21.3 (Pin_3), J21.5 (Pin_5), J9.1 (Pin_1), J9.3 (Pin_3), J9.5 (Pin_5), U12.5 (RESET), U12.6 (SLEEP), U13.5 (RESET), U13.6 (SLEEP), U14.5 (RESET), U14.6 (SLEEP), U15.5 (RESET), U15.6 (SLEEP), U16.5 (RESET), U16.6 (SLEEP), U17.5 (RESET), U17.6 (SLEEP)
- new net +VDC: U12.16 (VMOT), U13.16 (VMOT), U14.16 (VMOT), U15.16 (VMOT), U16.16 (VMOT), U17.16 (VMOT)
- new net E0DIR: J18.3 (Pin_3), U16.8 (DIR)
- new net E0ENABLE: J18.1 (Pin_1), U16.1 (ENABLE)
- new net E0STEP: J18.2 (Pin_2), U16.7 (STEP)
- new net E1DIR: J19.3 (Pin_3), U17.8 (DIR)
- new net E1ENABLE: J19.1 (Pin_1), U17.1 (ENABLE)
- new net E1STEP: J19.2 (Pin_2), U17.7 (STEP)
- new net GND: J18.4 (Pin_4), J19.4 (Pin_4), J6.4 (Pin_4), J7.4 (Pin_4), J8.4 (Pin_4), U12.15 (GND), U12.9 (GND), U13.15 (GND), U13.9 (GND), U14.15 (GND), U14.9 (GND), U15.15 (GND), U15.9 (GND), U16.15 (GND), U16.9 (GND), U17.15 (GND), U17.9 (GND)
- new net XDIR: J6.1 (Pin_1), U12.8 (DIR)
- new net XENABLE: J6.3 (Pin_3), U12.1 (ENABLE)
- new net XSTEP: J6.2 (Pin_2), U12.7 (STEP)
- new net YDIR: J7.1 (Pin_1), U13.8 (DIR)
- new net YENABLE: J7.3 (Pin_3), U13.1 (ENABLE)
- new net YSTEP: J7.2 (Pin_2), U13.7 (STEP)
- new net ZDIR: J8.1 (Pin_1), U14.8 (DIR)
- new net ZENABLE: J8.3 (Pin_3), U14.1 (ENABLE), U15.1 (ENABLE)
- new net ZSTEP: J8.2 (Pin_2), U14.7 (STEP), U15.7 (STEP)
- no-connect marks 0 -> 2
Other:
- note added: "4 x TMC262 Trinamic Controllers for X, Y and Z \n2x DRV8825 TI Controllers for E0 and E1\n"

Commit message: Updated PCBS
Parts:
- removed J10, J11, J9: Conn_02x03_Odd_Even, Pin_Headers:Pin_Header_Straight_2x03_Pitch1.27mm_SMD, symbol Conn_02x03_Odd_Even
- removed J20, J21: Conn_02x03_Odd_Even, symbol Conn_02x03_Odd_Even
- added JP1, JP10, JP11, JP12, JP13, JP14, JP15, JP2, JP3, JP4, JP5, JP6, JP7, JP8, JP9: Jumper_NO_Small, Resistors_SMD:R_0402, symbol Jumper_NO_Small
- J12, J13, J14, J15, J16, J17: footprint Socket_Strips:Socket_Strip_Straight_1x04_Pitch2.54mm -> Connectors_Molex:Molex_KK-41791-04_04x3.96mm_Straight
Connections:
- net +3V3: now also JP1.1, JP10.1, JP11.1, JP12.1, JP13.1, JP14.1, JP15.1, JP2.1, JP3.1, JP4.1, JP5.1, JP6.1, JP7.1, JP8.1, JP9.1
- net at U12.2 (M0): now also JP4.2
- net at U12.3 (M1): now also JP5.2
- net at U12.4 (M2): now also JP6.2
- net at U13.2 (M0): now also JP7.2
- net at U13.3 (M1): now also JP8.2
- net at U13.4 (M2): now also JP9.2
- net at U14.2 (M0), U15.2 (M0): now also JP1.2
- net at U14.3 (M1), U15.3 (M1): now also JP2.2
- net at U14.4 (M2), U15.4 (M2): now also JP3.2
- net at U16.2 (M0): now also JP10.2
- net at U16.3 (M1): now also JP11.2
- net at U16.4 (M2): now also JP12.2
- net at U17.2 (M0): now also JP13.2
- net at U17.3 (M1): now also JP14.2
- net at U17.4 (M2): now also JP15.2
- net +VDC renamed VAA

Commit message: Added routed Power switching circuitry
Parts:
- removed J12, J13, J14, J15, J16, J17: Conn_01x04, Connectors_Molex:Molex_KK-41791-04_04x3.96mm_Straight, symbol Conn_01x04
- removed JP1, JP10, JP11, JP12, JP13, JP14, JP15, JP2, JP3, JP4, JP5, JP6, JP7, JP8, JP9: Jumper_NO_Small, Resistors_SMD:R_0402, symbol Jumper_NO_Small
- removed U12, U13, U14, U15, U16, U17: pololu_DRV8825, .pretty:DRV8825, symbol pololu_DRV8825
- added J1, J12, J13, J14, J15, J2: Conn_01x03, Connectors_Molex:Molex_KK-6410-03_03x2.54mm_Straight, symbol Connector_Generic:Conn_01x03
- J18, J19, J6, J7, J8: footprint Socket_Strips:Socket_Strip_Straight_1x04_Pitch2.54mm -> Connectors_Molex:Molex_KK-6410-04_04x2.54mm_Straight; symbol Conn_01x04 -> PrinterController-rescue:Conn_01x04
Connections:
- net +3V3: now also J1.2 (Pin_2), J12.2 (Pin_2), J13.2 (Pin_2), J14.2 (Pin_2), J15.2 (Pin_2), J2.2 (Pin_2)
- net GND: now also J1.1 (Pin_1), J12.1 (Pin_1), J13.1 (Pin_1), J14.1 (Pin_1), J15.1 (Pin_1), J2.1 (Pin_1)
- net XDIR: now also J6.3 (Pin_3); no longer J6.1 (Pin_1)
- net XENABLE: now also J6.1 (Pin_1); no longer J6.3 (Pin_3)
- net YDIR: now also J7.3 (Pin_3); no longer J7.1 (Pin_1)
- net YENABLE: now also J7.1 (Pin_1); no longer J7.3 (Pin_3)
- net ZDIR: now also J8.3 (Pin_3); no longer J8.1 (Pin_1)
- net ZENABLE: now also J8.1 (Pin_1); no longer J8.3 (Pin_3)
- new net ESX1: J1.3 (Pin_3)
- new net ESX2: J13.3 (Pin_3)
- new net ESY1: J2.3 (Pin_3)
- new net ESY2: J14.3 (Pin_3)
- new net ESZ1: J12.3 (Pin_3)
- new net ESZ2: J15.3 (Pin_3)
- no-connect marks 2 -> 0
Other:
- note removed: "4 x TMC262 Trinamic Controllers for X, Y and Z \n2x DRV8825 TI Controllers for E0 and E1\n"
- moved on the sheet: J18, J19, J6, J7, J8

Commit message: Added updates to controller hardware
Parts:
- added J26: Conn_01x06, Connectors_JST:JST_EH_B06B-EH-A_06x2.50mm_Straight, symbol Connector_Generic:Conn_01x06
- J1, J12, J13, J14, J15, J2: footprint Connectors_Molex:Molex_KK-6410-03_03x2.54mm_Straight -> Connectors_JST:JST_EH_B03B-EH-A_03x2.50mm_Straight
- J18, J19, J6, J7, J8: footprint Connectors_Molex:Molex_KK-6410-04_04x2.54mm_Straight -> Connectors_JST:JST_EH_B04B-EH-A_04x2.50mm_Straight
Connections:
- wire segments 55 -> 84
Changed lines of the file:
@@
 F 0 "J6" H 2050 1950 50  0000 C CNN
 F 1 "Conn_01x04" H 2050 1450 50  0000 C CNN
-F 2 "Connectors_Molex:Molex_KK-6410-04_04x2.54mm_Straight" H 2050 1750 50  0001 C CNN
+F 2 "Connectors_JST:JST_EH_B04B-EH-A_04x2.50mm_Straight" H 2050 1750 50  0001 C CNN
 F 3 "" H 2050 1750 50  0001 C CNN
 	1    2050 1750
@@
 F 0 "J7" H 2050 2650 50  0000 C CNN
 F 1 "Conn_01x04" H 2050 2150 50  0000 C CNN
-F 2 "Connectors_Molex:Molex_KK-6410-04_04x2.54mm_Straight" H 2050 2450 50  0001 C CNN
+F 2 "Connectors_JST:JST_EH_B04B-EH-A_04x2.50mm_Straight" H 2050 2450 50  0001 C CNN
 F 3 "" H 2050 2450 50  0001 C CNN
 	1    2050 2450
@@
 F 0 "J18" H 2050 4050 50  0000 C CNN
 F 1 "Conn_01x04" H 2050 3550 50  0000 C CNN
-F 2 "Connectors_Molex:Molex_KK-6410-04_04x2.54mm_Straight" H 2050 3850 50  0001 C CNN
+F 2 "Connectors_JST:JST_EH_B04B-EH-A_04x2.50mm_Straight" H 2050 3850 50  0001 C CNN
 F 3 "" H 2050 3850 50  0001 C CNN
 	1    2050 3850
@@
 F 0 "J19" H 2050 4650 50  0000 C CNN
 F 1 "Conn_01x04" H 2050 4150 50  0000 C CNN
-F 2 "Connectors_Molex:Molex_KK-6410-04_04x2.54mm_Straight" H 2050 4450 50  0001 C CNN
+F 2 "Connectors_JST:JST_EH_B04B-EH-A_04x2.50mm_Straight" H 2050 4450 50  0001 C CNN
 F 3 "" H 2050 4450 50  0001 C CNN
 	1    2050 4450
@@
 F 0 "J8" H 2050 3250 50  0000 C CNN
 F 1 "Conn_01x04" H 2050 2750 50  0000 C CNN
-F 2 "Connectors_Molex:Molex_KK-6410-04_04x2.54mm_Straight" H 2050 3050 50  0001 C CNN
+F 2 "Connectors_JST:JST_EH_B04B-EH-A_04x2.50mm_Straight" H 2050 3050 50  0001 C CNN
 F 3 "" H 2050 3050 50  0001 C CNN
 	1    2050 3050
@@
 F 0 "J1" H 2030 5442 50  0000 L CNN
 F 1 "Conn_01x03" H 2030 5351 50  0000 L CNN
-F 2 "Connectors_Molex:Molex_KK-6410-03_03x2.54mm_Straight" H 1950 5400 50  0001 C CNN
+F 2 "Connectors_JST:JST_EH_B03B-EH-A_03x2.50mm_Straight" H 1950 5400 50  0001 C CNN
 F 3 "~" H 1950 5400 50  0001 C CNN
 	1    1950 5400
@@
 F 0 "J2" H 2030 5842 50  0000 L CNN
 F 1 "Conn_01x03" H 2030 5751 50  0000 L CNN
-F 2 "Connectors_Molex:Molex_KK-6410-03_03x2.54mm_Straight" H 1950 5800 50  0001 C CNN
+F 2 "Connectors_JST:JST_EH_B03B-EH-A_03x2.50mm_Straight" H 1950 5800 50  0001 C CNN
 F 3 "~" H 1950 5800 50  0001 C CNN
 	1    1950 5800
@@
 F 0 "J12" H 2030 6242 50  0000 L CNN
 F 1 "Conn_01x03" H 2030 6151 50  0000 L CNN
-F 2 "Connectors_Molex:Molex_KK-6410-03_03x2.54mm_Straight" H 1950 6200 50  0001 C CNN
+F 2 "Connectors_JST:JST_EH_B03B-EH-A_03x2.50mm_Straight" H 1950 6200 50  0001 C CNN
 F 3 "~" H 1950 6200 50  0001 C CNN
 	1    1950 6200
@@
 F 0 "J13" H 2030 6692 50  0000 L CNN
 F 1 "Conn_01x03" H 2030 6601 50  0000 L CNN
-F 2 "Connectors_Molex:Molex_KK-6410-03_03x2.54mm_Straight" H 1950 6650 50  0001 C CNN
+F 2 "Connectors_JST:JST_EH_B03B-EH-A_03x2.50mm_Straight" H 1950 6650 50  0001 C CNN
 F 3 "~" H 1950 6650 50  0001 C CNN
 	1    1950 6650
@@
 F 0 "J14" H 2030 7092 50  0000 L CNN
 F 1 "Conn_01x03" H 2030 7001 50  0000 L CNN
-F 2 "Connectors_Molex:Molex_KK-6410-03_03x2.54mm_Straight" H 1950 7050 50  0001 C CNN
+F 2 "Connectors_JST:JST_EH_B03B-EH-A_03x2.50mm_Straight" H 1950 7050 50  0001 C CNN
 F 3 "~" H 1950 7050 50  0001 C CNN
 	1    1950 7050
@@
 F 0 "J15" H 2030 7492 50  0000 L CNN
 F 1 "Conn_01x03" H 2030 7401 50  0000 L CNN
-F 2 "Connectors_Molex:Molex_KK-6410-03_03x2.54mm_Straight" H 1950 7450 50  0001 C CNN
+F 2 "Connectors_JST:JST_EH_B03B-EH-A_03x2.50mm_Straight" H 1950 7450 50  0001 C CNN
 F 3 "~" H 1950 7450 50  0001 C CNN
 	1    1950 7450
@@
 ESZ2
 Wire Wire Line
-	1750 7550 1300 7550
-Wire Wire Line
-	1750 7150 1300 7150
-Wire Wire Line
-	1750 6750 1300 6750
-Wire Wire Line
-	1750 6300 1300 6300
-Wire Wire Line
-	1300 5900 1750 5900
-Wire Wire Line
-	1750 5500 1300 5500
+	1750 7550 1700 7550
+Wire Wire Line
+	1750 7150 1700 7150
+Wire Wire Line
+	1750 6750 1700 6750
+Wire Wire Line
+	1750 6300 1700 6300
+Wire Wire Line
+	1300 5900 1700 5900
+Wire Wire Line
+	1750 5500 1700 5500
 Wire Wire Line
 	1750 7450 1500 7450
@@
 	1    0    0    -1
 $EndComp
+$Comp
+L Connector_Generic:Conn_01x06 J26
+U 1 1 5B7315D5
+P 3100 5950
+F 0 "J26" H 3180 5942 50  0000 L CNN
+F 1 "Conn_01x06" H 3180 5851 50  0000 L CNN
+F 2 "Connectors_JST:JST_EH_B06B-EH-A_06x2.50mm_Straight" H 3100 5950 50  0001 C CNN
+F 3 "~" H 3100 5950 50  0001 C CNN
+	1    3100 5950
+	1    0    0    -1
+$EndComp
+Wire Wire Line
+	1700 5500 1700 5600
+Wire Wire Line
+	1700 5600 2900 5600
+Wire Wire Line
+	2900 5600 2900 5750
+Connection ~ 1700 5500
+Wire Wire Line
+	1700 5500 1300 5500
+Wire Wire Line
+	2900 5850 2500 5850
+Wire Wire Line
+	2500 5850 2500 6000
+Wire Wire Line
+	2500 6000 1700 6000
+Wire Wire Line
+	1700 6000 1700 5900
+Connection ~ 1700 5900
+Wire Wire Line
+	1700 5900 1750 5900
+Wire Wire Line
+	1700 6300 1700 6400
+Wire Wire Line
+	1700 6400 2550 6400
+Wire Wire Line
+	2550 6400 2550 5950
+Wire Wire Line
+	2550 5950 2900 5950
+Connection ~ 1700 6300
+Wire Wire Line
+	1700 6300 1300 6300
+Wire Wire Line
+	2900 6050 2600 6050
+Wire Wire Line
+	2600 6050 2600 6850
+Wire Wire Line
+	2600 6850 1700 6850
+Wire Wire Line
+	1700 6850 1700 6750
+Connection ~ 1700 6750
+Wire Wire Line
+	1700 6750 1300 6750
+Wire Wire Line
+	2650 6150 2650 7250
+Wire Wire Line
+	2650 7250 1700 7250
+Wire Wire Line
+	1700 7250 1700 7150
+Wire Wire Line
+	2650 6150 2900 6150
+Connection ~ 1700 7150
+Wire Wire Line
+	1700 7150 1300 7150
+Wire Wire Line
+	2900 6250 2700 6250
+Wire Wire Line
+	2700 6250 2700 7650
+Wire Wire Line
+	2700 7650 1700 7650
+Wire Wire Line
+	1700 7650 1700 7550
+Connection ~ 1700 7550
+Wire Wire Line
+	1700 7550 1300 7550
 $EndSCHEMATC
