File: Hardware/Controllerv1/PrinterController/PrinterController.kicad_pcb (KiCad board)
At the start: 2 copper layers, 100 x 100 mm, 108 parts, among them J1 Conn_01x03, J10 Screw_Terminal_01x02, J11 Screw_Terminal_01x02, J12 Conn_01x03, J13 Conn_01x03, J14 Conn_01x03, J15 Conn_01x03, J16 Conn_01x02, J17 Conn_01x02, J18 Conn_01x04, J19 Conn_01x04, J2 Conn_01x03, J20 Conn_01x02, J21 USB_OTG, J22 Screw_Terminal_01x02, J23 Conn_01x03, J24 Screw_Terminal_01x02, J25 Conn_ARM_JTAG_SWD_10, J3 Conn_01x03, J4 Conn_01x03, J5 Screw_Terminal_01x02, J6 Conn_01x04, J7 Conn_01x04, J8 Conn_01x04, J9 Screw_Terminal_01x02, Q5 Q_NMOS_DGS, Q6 Q_NMOS_DGS, U1 R-78E5.0-1.0, U10 IRFR3711TRPBF, U11 IRFR3711TRPBF, U13 MCU-ATSAM3X8EA-AU-ND(LQFP144), U2 ZXGD3003E6, U3 ZXGD3003E6, U4 ZXGD3003E6, U5 ZXGD3003E6, U6 R-78E3.3-1.0, U8 IRFR3711TRPBF, U9 IRFR3711TRPBF, Y1 Crystal_GND24, Y2 32.768

Commit message: Added updates to controller hardware
Parts:
- added D2: LED, Diodes_SMD:D_0805, F.Cu at (188.1, 107.2)
- added D3: LED, Diodes_SMD:D_0805, F.Cu at (189.9, 107.2)
- added D6: LED, Diodes_SMD:D_0805, F.Cu at (192.5, 75.0)
- added J26: Conn_01x06, Connectors_JST:JST_EH_B06B-EH-A_06x2.50mm_Straight, F.Cu at (225.7, 77.5)
- added R16: 330R, Resistors_SMD:R_0805, F.Cu at (188.1, 110.6)
- added R18: 330R, Resistors_SMD:R_0805, F.Cu at (190.0, 110.6)
- added R19: 330R, Resistors_SMD:R_0805, F.Cu at (191.6, 72.3)
- added R20: 330R, Resistors_SMD:R_0805, F.Cu at (219.8, 106.9)
- C11, C5, L2, R4, R5: moved to B.Cu
- C27, C28, C29, C30, C31, C32: footprint Capacitors_Tantalum_SMD:CP_Tantalum_Case-A_EIA-3216-18_Hand -> Capacitors_SMD:CP_Elec_6.3x5.3
- C34, C38: footprint Capacitors_Tantalum_SMD:CP_Tantalum_Case-D_EIA-7343-31_Hand -> Capacitors_SMD:CP_Elec_6.3x7.7
- C35, C39: footprint Capacitors_Tantalum_SMD:CP_Tantalum_Case-D_EIA-7343-31_Hand -> Capacitors_SMD:CP_Elec_8x10
- C36, C40: footprint Capacitors_Tantalum_SMD:CP_Tantalum_Case-B_EIA-3528-21_Hand -> Capacitors_SMD:CP_Elec_6.3x7.7
- D1: footprint Capacitors_Tantalum_SMD:CP_Tantalum_Case-B_EIA-3528-21_Hand -> Diodes_SMD:D_0805
- J1, J12, J13, J14, J15, J2: footprint Connectors_Molex:Molex_KK-6410-03_03x2.54mm_Straight -> Connectors_JST:JST_EH_B03B-EH-A_03x2.50mm_Straight
- J16, J17, J20: footprint Connectors_Molex:Molex_KK-6410-02_02x2.54mm_Straight -> Connectors_JST:JST_EH_B02B-EH-A_02x2.50mm_Straight
- J18, J19, J6, J7, J8: footprint Connectors_Molex:Molex_KK-6410-04_04x2.54mm_Straight -> Connectors_JST:JST_EH_B04B-EH-A_04x2.50mm_Straight
- moved J21 95.5 mm to (236.1, 108.3), turned to 90 degrees
- moved C1 80.7 mm to (213.5, 106.5)
- moved L2 77.4 mm to (202.8, 97.3), turned to 270 degrees
- moved C11 76.0 mm to (204.7, 97.3), turned to 270 degrees
- moved C17 74.5 mm to (206.5, 73.8), turned to 90 degrees
- moved C2 74.2 mm to (211.7, 102.0)
- moved L3 69.5 mm to (202.6, 73.9), turned to 90 degrees
- moved L1 57.1 mm to (200.5, 73.9), turned to 90 degrees
- moved C23 54.6 mm to (198.5, 73.9), turned to 90 degrees
- moved C3 53.5 mm to (214.9, 88.9), turned to 90 degrees
- moved R2 52.9 mm to (204.5, 97.5), turned to 270 degrees
- moved C26 52.0 mm to (196.6, 73.9), turned to 90 degrees
- moved C4 45.4 mm to (214.9, 94.1)
- moved R3 43.2 mm to (202.5, 97.5), turned to 270 degrees
- moved R4 41.3 mm to (196.2, 91.4)
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Connections:
- U13 pad 23: (no net) -> Net-(D2-Pad2)
- U13 pad 24: (no net) -> Net-(D3-Pad2)
- U13 pad 85: (no net) -> Net-(D6-Pad2)
Routing:
- net +3V3: track 17.0 -> 323.4 mm, vias 0 -> 8
- net /Microcontroller/E0DIR: track 0.00 -> 110.4 mm, vias 0 -> 5
- net VDD: track 0.00 -> 108.1 mm, vias 0 -> 7
- net /Microcontroller/ZDIR: track 0.00 -> 78.2 mm, vias 0 -> 4
- net /DriverStage/HEATER3: track 14.7 -> 92.5 mm, vias 0 -> 1
- net +5V: track 54.0 -> 128.9 mm
- net /Motor Connections/ESX1: track 0.00 -> 73.6 mm, vias 0 -> 1
- net /Microcontroller/E0STEP: track 0.00 -> 71.1 mm, vias 0 -> 1
- net /Motor Connections/ESY1: track 0.00 -> 68.7 mm, vias 0 -> 1
- net /Microcontroller/TEMP3: track 0.00 -> 66.4 mm, vias 0 -> 4
- net /Motor Connections/ESZ1: track 0.00 -> 63.2 mm, vias 0 -> 1
- net /DriverStage/FAN2: track 24.7 -> 86.6 mm, vias 1 -> 4
- net /Motor Connections/ESX2: track 0.00 -> 60.1 mm, vias 0 -> 1
- net /Microcontroller/TEMP2: track 0.00 -> 59.4 mm, vias 0 -> 4
- net /Microcontroller/TEMP1: track 0.00 -> 55.2 mm, vias 0 -> 4
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- added copper zone on B.Cu, net GND
- added copper zone on F.Cu, net GND
Other:
- net class Default: clearance 0.2 -> 0.16
- rule trace_clearance: 0.2 -> 0.16
