File: Hardware/Controllerv1/PrinterController/SensorInputs.sch (KiCad schematic (older format))
At the start: 0 parts

Commit message: Added routed Power switching circuitry
Parts:
- added J16, J17, J20: Conn_01x02, Connectors_Molex:Molex_KK-6410-02_02x2.54mm_Straight, symbol Connector_Generic:Conn_01x02
- added R25, R26, R27: 100K, Resistors_SMD:R_0805, symbol Device:R
Connections:
- net labels added: +3V3, GND, TEMP1, TEMP2, TEMP3
- wire segments 0 -> 19

Commit message: Added updates to controller hardware
Parts:
- J16, J17, J20: footprint Connectors_Molex:Molex_KK-6410-02_02x2.54mm_Straight -> Connectors_JST:JST_EH_B02B-EH-A_02x2.50mm_Straight
Changed lines of the file:
@@
 $Descr A4 11693 8268
 encoding utf-8
-Sheet 6 6
+Sheet 5 6
 Title ""
 Date ""
@@
 F 0 "J16" H 1870 975 50  0000 C CNN
 F 1 "Conn_01x02" H 1870 1066 50  0000 C CNN
-F 2 "Connectors_Molex:Molex_KK-6410-02_02x2.54mm_Straight" H 1950 1300 50  0001 C CNN
+F 2 "Connectors_JST:JST_EH_B02B-EH-A_02x2.50mm_Straight" H 1950 1300 50  0001 C CNN
 F 3 "~" H 1950 1300 50  0001 C CNN
 	1    1950 1300
@@
 F 0 "J17" H 1870 1425 50  0000 C CNN
 F 1 "Conn_01x02" H 1870 1516 50  0000 C CNN
-F 2 "Connectors_Molex:Molex_KK-6410-02_02x2.54mm_Straight" H 1950 1750 50  0001 C CNN
+F 2 "Connectors_JST:JST_EH_B02B-EH-A_02x2.50mm_Straight" H 1950 1750 50  0001 C CNN
 F 3 "~" H 1950 1750 50  0001 C CNN
 	1    1950 1750
@@
 F 0 "J20" H 1870 1925 50  0000 C CNN
 F 1 "Conn_01x02" H 1870 2016 50  0000 C CNN
-F 2 "Connectors_Molex:Molex_KK-6410-02_02x2.54mm_Straight" H 1950 2250 50  0001 C CNN
+F 2 "Connectors_JST:JST_EH_B02B-EH-A_02x2.50mm_Straight" H 1950 2250 50  0001 C CNN
 F 3 "~" H 1950 2250 50  0001 C CNN
 	1    1950 2250
