File: Hardware/Controllerv1/PrinterController/ATSAM3X8E.sch (KiCad schematic (older format))
At the start: 40 parts

Commit message: Added main controller and Power Outputs
Parts:
- added D1: LED, LEDs:LED_0805, symbol LED
- added R6: 330R, Resistors_SMD:R_0805, symbol R
- C1: renamed from C?; footprint (none) -> .pretty:SOT65P330X90-5N
- C10, C11, C12, C13, C14, C15, C16, C17, C18, C19, C2, C20, C21, C22, C23, C24, C25, C26, C3, C4, C5, C6, C7, C8, C9: renamed from C?; footprint (none) -> Capacitors_SMD:C_0805
- J1: renamed from J?; footprint (none) -> Connectors:USB_Micro-B_10103594-0001LF
- J2: renamed from J?; footprint Connector_PinHeader_1.27mm:PinHeader_2x05_P1.27mm_Vertical_SMD -> Pin_Headers:Pin_Header_Straight_2x05_Pitch1.27mm
- L1, L2, L3, L4: renamed from L?; footprint (none) -> Inductors_SMD:L_0805
- R1, R2, R3, R4, R5: renamed from R?; footprint (none) -> Resistors_SMD:R_0805
- Y1, Y2: renamed from Y?; footprint (none) -> Crystals:Crystal_HC52-8mm_Horizontal
- gave numbers to parts that had none: 1
Connections:
- net labels added: E0DIR, E0ENABLE, E0STEP, E1DIR, E1ENABLE, E1STEP, FAN1, FAN2, HEATER1, HEATER2, HEATER3, HEATER4, XDIR, XENABLE, XMAX, XMIN, XSTEP, YDIR, YENABLE, YMAX, YMIN, YSTEP, ZDIR, ZENABLE, ZMAX, ZMIN, ZSTEP
- net labels removed: FETOutputs
- wire segments 115 -> 109
Other:
- note removed: "FET Driven Outputs (4 x High Current + 2 x Fan outputs)\n"

Commit message: Added updates to PCB
Parts:
- U1: footprint LQFP144-0.5-20X20M -> MCU-ATSAM3X8EA-AU-ND_LQFP144_:LQFP144-0.5-20X20M
- Y1: footprint Crystals:Crystal_HC52-8mm_Horizontal -> Crystals:Crystal_SMD_HC49-SD_HandSoldering
- Y2: footprint Crystals:Crystal_HC52-8mm_Horizontal -> Crystals:Crystal_SMD_MicroCrystal_CC7V-T1A-2pin_3.2x1.5mm_HandSoldering
Changed lines of the file:
@@
 LIBS:zetex
 LIBS:Zilog
+LIBS:IRFR3711TRPBF
 LIBS:PrinterController-cache
 EELAYER 25 0
@@
 F 0 "Y2" V 904 2481 50  0000 L CNN
 F 1 "32.768" V 995 2481 50  0000 L CNN
-F 2 "Crystals:Crystal_HC52-8mm_Horizontal" H 950 2350 50  0001 C CNN
+F 2 "Crystals:Crystal_SMD_MicroCrystal_CC7V-T1A-2pin_3.2x1.5mm_HandSoldering" H 950 2350 50  0001 C CNN
 F 3 "~" H 950 2350 50  0001 C CNN
 	1    950  2350
@@
 F 0 "Y1" V 904 2131 50  0000 L CNN
 F 1 "12MHz" V 995 2131 50  0000 L CNN
-F 2 "Crystals:Crystal_HC52-8mm_Horizontal" H 950 2000 50  0001 C CNN
+F 2 "Crystals:Crystal_SMD_HC49-SD_HandSoldering" H 950 2000 50  0001 C CNN
 F 3 "~" H 950 2000 50  0001 C CNN
 	1    950  2000
@@
 F 0 "U1" H 4050 7028 50  0000 C CNN
 F 1 "MCU-ATSAM3X8EA-AU-ND(LQFP144)" H 4050 6937 50  0000 C CNN
-F 2 "LQFP144-0.5-20X20M" H 4050 4100 50  0001 L BNN
+F 2 "MCU-ATSAM3X8EA-AU-ND_LQFP144_:LQFP144-0.5-20X20M" H 4050 4100 50  0001 L BNN
 F 3 "Microchip" H 4050 4100 50  0001 L BNN
 F 4 "None" H 4050 4100 50  0001 L BNN "Field4"

Commit message: Updated PCBS
Parts:
- removed Y1: 12MHz, Crystals:Crystal_SMD_HC49-SD_HandSoldering, symbol Device:Crystal
- added Y1: Crystal_GND24, Crystals:Crystal_SMD_3225-4pin_3.2x2.5mm_HandSoldering, symbol Crystal_GND24
- C1: footprint .pretty:SOT65P330X90-5N -> Capacitors_SMD:C_0805
Connections:
- wire segments 109 -> 114
Changed lines of the file:
@@
 F 0 "C1" V 348 1650 50  0000 C CNN
 F 1 "C" V 439 1650 50  0000 C CNN
-F 2 ".pretty:SOT65P330X90-5N" H 638 1500 50  0001 C CNN
+F 2 "Capacitors_SMD:C_0805" H 638 1500 50  0001 C CNN
 F 3 "~" H 600 1650 50  0001 C CNN
 	1    600  1650
@@
 F 3 "~" H 950 2350 50  0001 C CNN
 	1    950  2350
-	0    1    1    0
-$EndComp
-$Comp
-L Device:Crystal Y1
-U 1 1 5B26AA8B
-P 950 2000
-F 0 "Y1" V 904 2131 50  0000 L CNN
-F 1 "12MHz" V 995 2131 50  0000 L CNN
-F 2 "Crystals:Crystal_SMD_HC49-SD_HandSoldering" H 950 2000 50  0001 C CNN
-F 3 "~" H 950 2000 50  0001 C CNN
-	1    950  2000
 	0    1    1    0
 $EndComp
@@
 	950  1650 750  1650
 Wire Wire Line
-	950  1850 950  1650
-Wire Wire Line
 	750  2150 750  2050
 Wire Wire Line
@@
 Connection ~ 500  2500
 Wire Wire Line
-	450  2250 450  1650
+	450  2250 450  1550
 Connection ~ 450  2050
 Connection ~ 500  2250
@@
 	1200 2250 1700 2250
 Wire Wire Line
-	1200 2050 1700 2050
-Wire Wire Line
-	1200 2150 1200 2050
-Wire Wire Line
-	1200 1850 950  1850
-Wire Wire Line
-	1200 1950 1200 1850
+	1150 2050 1700 2050
 Wire Wire Line
 	1700 1950 1200 1950
@@
 	800  2200 1200 2200
 Connection ~ 950  2200
-Wire Wire Line
-	750  2150 1200 2150
-Connection ~ 950  2150
-Connection ~ 950  1850
 Wire Wire Line
 	2800 1150 2800 1350
@@
 	1    0    0    -1
 $EndComp
+$Comp
+L Crystal_GND24 Y1
+U 1 1 5B358941
+P 950 2000
+F 0 "Y1" H 1075 2200 50  0000 L CNN
+F 1 "Crystal_GND24" H 1075 2125 50  0000 L CNN
+F 2 "Crystals:Crystal_SMD_3225-4pin_3.2x2.5mm_HandSoldering" H 950 2000 50  0001 C CNN
+F 3 "" H 950 2000 50  0001 C CNN
+	1    950  2000
+	0    1    1    0
+$EndComp
+Wire Wire Line
+	1150 2150 1150 2050
+Wire Wire Line
+	750  2150 1150 2150
+Connection ~ 950  2150
+Wire Wire Line
+	1200 1950 1200 1850
+Wire Wire Line
+	1200 1850 950  1850
+Wire Wire Line
+	950  1850 950  1650
+Wire Wire Line
+	1150 2000 1300 2000
+Wire Wire Line
+	1300 2000 1300 1550
+Wire Wire Line
+	1300 1550 450  1550
+Connection ~ 450  1650
+Wire Wire Line
+	750  2000 750  1850
+Wire Wire Line
+	750  1850 450  1850
+Connection ~ 450  1850
 $EndSCHEMATC

Commit message: Added routed Power switching circuitry
Parts:
- removed J1: USB_B_Micro, Connectors:USB_Micro-B_10103594-0001LF, symbol Connector_Specialized:USB_B_Micro
- removed J2: Conn_ARM_JTAG_SWD_10, Pin_Headers:Pin_Header_Straight_2x05_Pitch1.27mm, symbol Connector_Specialized:Conn_ARM_JTAG_SWD_10
- removed U1: MCU-ATSAM3X8EA-AU-ND(LQFP144), MCU-ATSAM3X8EA-AU-ND_LQFP144_:LQFP144-0.5-20X20M, symbol MCU-ATSAM3X8EA-AU-ND_LQFP144_:MCU-ATSAM3X8EA-AU-ND(LQFP144)
- added J21: USB_OTG, Connectors_USB:USB_Micro-B_Molex-105017-0001, symbol Connector:USB_OTG
- added J25: Conn_ARM_JTAG_SWD_10, Connectors_Harwin:Harwin_Gecko-G125-FVX1005L0X_2x05x1.25mm_Straight, symbol Connector:Conn_ARM_JTAG_SWD_10
- added U13: MCU-ATSAM3X8EA-AU-ND(LQFP144), MCU-ATSAM3X8EA-AU-ND_LQFP144_:LQFP144-0.5-20X20M, symbol MCU-ATSAM3X8EA-AU-ND_LQFP144_:MCU-ATSAM3X8EA-AU-ND(LQFP144)
- D1: footprint LEDs:LED_0805 -> Capacitors_Tantalum_SMD:CP_Tantalum_Case-B_EIA-3528-21_Hand; symbol LED -> PrinterController-rescue:LED
- R6: symbol R -> PrinterController-rescue:R
- Y1: symbol Crystal_GND24 -> PrinterController-rescue:Crystal_GND24
Connections:
- net labels added: TEMP1, TEMP2, TEMP3
- wire segments 114 -> 130
Changed lines of the file:
@@
-EESchema Schematic File Version 2
-LIBS:74xgxx
-LIBS:74xx
-LIBS:ac-dc
-LIBS:actel
-LIBS:adc-dac
-LIBS:allegro
-LIBS:Altera
-LIBS:analog_devices
-LIBS:analog_switches
-LIBS:atmel
-LIBS:audio
-LIBS:battery_management
-LIBS:bbd
-LIBS:bosch
-LIBS:brooktre
-LIBS:cmos_ieee
-LIBS:cmos4000
-LIBS:conn
-LIBS:contrib
-LIBS:cypress
-LIBS:dc-dc
-LIBS:device
-LIBS:digital-audio
-LIBS:diode
-LIBS:display
-LIBS:dsp
-LIBS:elec-unifil
-LIBS:ESD_Protection
-LIBS:ftdi
-LIBS:gennum
-LIBS:graphic_symbols
-LIBS:hc11
-LIBS:infineon
-LIBS:intel
-LIBS:interface
-LIBS:intersil
-LIBS:ir
-LIBS:Lattice
-LIBS:leds
-LIBS:LEM
-LIBS:linear
-LIBS:logic_programmable
-LIBS:maxim
-LIBS:mechanical
-LIBS:memory
-LIBS:microchip
-LIBS:microchip_dspic33dsc
-LIBS:microchip_pic10mcu
-LIBS:microchip_pic12mcu
-LIBS:microchip_pic16mcu
-LIBS:microchip_pic18mcu
-LIBS:microchip_pic24mcu
-LIBS:microchip_pic32mcu
-LIBS:microcontrollers
-LIBS:modules
-LIBS:motor_drivers
-LIBS:motorola
-LIBS:motors
-LIBS:msp430
-LIBS:nordicsemi
-LIBS:nxp
-LIBS:nxp_armmcu
-LIBS:onsemi
-LIBS:opto
-LIBS:Oscillators
-LIBS:philips
-LIBS:power
-LIBS:Power_Management
-LIBS:powerint
-LIBS:pspice
-LIBS:references
-LIBS:regul
-LIBS:relays
-LIBS:rfcom
-LIBS:RFSolutions
-LIBS:sensors
-LIBS:silabs
-LIBS:siliconi
-LIBS:stm8
-LIBS:stm32
-LIBS:supertex
-LIBS:switches
-LIBS:texas
-LIBS:transf
-LIBS:transistors
-LIBS:triac_thyristor
-LIBS:ttl_ieee
-LIBS:valves
-LIBS:video
-LIBS:wiznet
-LIBS:Worldsemi
-LIBS:Xicor
-LIBS:xilinx
-LIBS:zetex
-LIBS:Zilog
-LIBS:IRFR3711TRPBF
+EESchema Schematic File Version 4
 LIBS:PrinterController-cache
-EELAYER 25 0
+EELAYER 26 0
 EELAYER END
 $Descr A4 11693 8268
 encoding utf-8
-Sheet 2 6
+Sheet 6 6
 Title ""
 Date ""
@@
 	1    5400 850
 	0    1    1    0
-$EndComp
-$Comp
-L MCU-ATSAM3X8EA-AU-ND_LQFP144_:MCU-ATSAM3X8EA-AU-ND(LQFP144) U?
-U 1 1 5B26AB43
-P 4050 4100
-AR Path="/5B26AB43" Ref="U?"  Part="1"
-AR Path="/5B2631DE/5B26AB43" Ref="U1"  Part="1"
-F 0 "U1" H 4050 7028 50  0000 C CNN
-F 1 "MCU-ATSAM3X8EA-AU-ND(LQFP144)" H 4050 6937 50  0000 C CNN
-F 2 "MCU-ATSAM3X8EA-AU-ND_LQFP144_:LQFP144-0.5-20X20M" H 4050 4100 50  0001 L BNN
-F 3 "Microchip" H 4050 4100 50  0001 L BNN
-F 4 "None" H 4050 4100 50  0001 L BNN "Field4"
-F 5 "None" H 4050 4100 50  0001 L BNN "Field5"
-F 6 "Unavailable" H 4050 4100 50  0001 L BNN "Field6"
-F 7 "SMD IC MCU 32BIT 512KB FLASH 84MHz" H 4050 4100 50  0001 L BNN "Field7"
-F 8 "ATSAM3X8EA-AU-ND" H 4050 4100 50  0001 L BNN "Field8"
-	1    4050 4100
-	1    0    0    -1
-$EndComp
-$Comp
-L Connector_Specialized:Conn_ARM_JTAG_SWD_10 J2
-U 1 1 5B26C706
-P 6450 7200
-F 0 "J2" H 6009 7154 50  0000 R CNN
-F 1 "Conn_ARM_JTAG_SWD_10" H 6009 7245 50  0000 R CNN
-F 2 "Pin_Headers:Pin_Header_Straight_2x05_Pitch1.27mm" H 6500 6650 50  0001 L TNN
-F 3 "http://infocenter.arm.com/help/topic/com.arm.doc.faqs/attached/13634/cortex_debug_connectors.pdf" V 6100 5950 50  0001 C CNN
-	1    6450 7200
-	-1   0    0    1
 $EndComp
 Text Label 5650 7500 0    50   ~ 0
@@
 VDDREF
 $Comp
-L Connector_Specialized:USB_B_Micro J1
-U 1 1 5B29302C
-P 700 3750
-F 0 "J1" H 755 4217 50  0000 C CNN
-F 1 "USB_B_Micro" H 755 4126 50  0000 C CNN
-F 2 "Connectors:USB_Micro-B_10103594-0001LF" H 850 3700 50  0001 C CNN
-F 3 "~" H 850 3700 50  0001 C CNN
-	1    700  3750
-	1    0    0    -1
-$EndComp
-$Comp
 L power:VBUS #PWR046
 U 1 1 5B297F54
@@
 $EndComp
 Wire Wire Line
-	1350 3300 1650 3300
+	1350 3300 1500 3300
 Connection ~ 1500 3300
 Wire Wire Line
-	1350 2950 1700 2950
+	1350 2950 1650 2950
 Wire Wire Line
 	1650 3000 1650 2950
@@
 Connection ~ 500  2500
 Wire Wire Line
-	450  2250 450  1550
+	450  2250 450  2050
 Connection ~ 450  2050
 Connection ~ 500  2250
@@
 	1700 1950 1200 1950
 Wire Wire Line
-	800  2500 1200 2500
+	800  2500 950  2500
 Connection ~ 950  2500
 Wire Wire Line
-	800  2200 1200 2200
+	800  2200 950  2200
 Connection ~ 950  2200
 Wire Wire Line
@@
 	2800 800  2800 850
 Wire Wire Line
-	3400 950  3650 950
+	3400 950  3600 950
 Wire Wire Line
 	3400 1350 3400 1250
@@
 	4300 1100 4300 1350
 Wire Wire Line
-	3600 700  3600 1350
+	3600 700  3600 950
 Connection ~ 3600 950
 Connection ~ 3600 700
@@
 	4600 850  4600 1350
 Wire Wire Line
-	4600 850  5250 850
+	4600 850  4900 850
 Connection ~ 4900 850
 Wire Wire Line
 	4900 1350 4900 850
 Wire Wire Line
-	5750 650  6600 650
+	5750 650  5950 650
 Connection ~ 6350 650
 Connection ~ 5950 650
 Wire Wire Line
-	3600 1350 4000 1350
-Connection ~ 3900 1350
-Connection ~ 3800 1350
-Connection ~ 3700 1350
-Connection ~ 3600 1350
-Wire Wire Line
-	4900 1350 5300 1350
-Connection ~ 5200 1350
-Connection ~ 5100 1350
-Connection ~ 5000 1350
-Connection ~ 4900 1350
-Wire Wire Line
-	5500 1350 6400 1350
-Connection ~ 5800 1350
-Connection ~ 5600 1350
-Connection ~ 5700 1350
-Connection ~ 6400 2050
-Wire Wire Line
-	6400 1350 6400 2050
-Connection ~ 6400 1950
-Connection ~ 6400 1850
-Connection ~ 6400 1750
-Wire Wire Line
 	5950 7200 5700 7200
 Wire Wire Line
@@
 	5950 7500 5650 7500
 Wire Wire Line
-	6450 6600 6550 6600
+	6450 6600 6500 6600
 Wire Wire Line
 	6650 6500 6500 6500
@@
 Wire Wire Line
 	1100 2650 1250 2650
-Wire Wire Line
-	700  4150 600  4150
-Connection ~ 700  4150
 Text HLabel 4700 7300 3    60   Output ~ 0
 ZSTEP
@@
 	5300 6850 5300 7350
 $Comp
-L LED D1
+L PrinterController-rescue:LED D1
 U 1 1 5B238618
 P 5400 7500
 F 0 "D1" H 5400 7600 50  0000 C CNN
 F 1 "LED" H 5400 7400 50  0000 C CNN
-F 2 "LEDs:LED_0805" H 5400 7500 50  0001 C CNN
+F 2 "Capacitors_Tantalum_SMD:CP_Tantalum_Case-B_EIA-3528-21_Hand" H 5400 7500 50  0001 C CNN
 F 3 "" H 5400 7500 50  0001 C CNN
 	1    5400 7500
@@
 	5300 7350 5400 7350
 $Comp
-L R R6
+L PrinterController-rescue:R R6
 U 1 1 5B23892D
 P 5250 7700
@@
 $EndComp
 $Comp
-L Crystal_GND24 Y1
+L PrinterController-rescue:Crystal_GND24 Y1
 U 1 1 5B358941
 P 950 2000
@@
 	1150 2150 1150 2050
 Wire Wire Line
-	750  2150 1150 2150
+	750  2150 950  2150
 Connection ~ 950  2150
 Wire Wire Line
@@
 	750  1850 450  1850
 Connection ~ 450  1850
+Wire Wire Line
+	1500 3300 1650 3300
+Wire Wire Line
+	1650 2950 1700 2950
+Wire Wire Line
+	450  2050 450  1850
+Wire Wire Line
+	950  2500 1200 2500
+Wire Wire Line
+	950  2200 1200 2200
+Wire Wire Line
+	3600 950  3650 950
+Wire Wire Line
+	3600 950  3600 1100
+Wire Wire Line
+	3600 1100 3600 1350
+Wire Wire Line
+	4900 850  5250 850
+Wire Wire Line
+	6350 650  6600 650
+Wire Wire Line
+	5950 650  6350 650
+Wire Wire Line
+	6500 6600 6550 6600
+Wire Wire Line
+	950  2150 1150 2150
+Wire Wire Line
+	450  1650 450  1550
+Wire Wire Line
+	450  1850 450  1650
+Wire Wire Line
+	6400 1350 6400 1750
+$Comp
+L MCU-ATSAM3X8EA-AU-ND_LQFP144_:MCU-ATSAM3X8EA-AU-ND(LQFP144) U13
+U 1 1 5B6CC3DF
+P 4050 4100
+F 0 "U13" H 4050 7028 50  0000 C CNN
+F 1 "MCU-ATSAM3X8EA-AU-ND(LQFP144)" H 4050 6937 50  0000 C CNN
+F 2 "MCU-ATSAM3X8EA-AU-ND_LQFP144_:LQFP144-0.5-20X20M" H 4050 4100 50  0001 L BNN
+F 3 "Microchip" H 4050 4100 50  0001 L BNN
+F 4 "None" H 4050 4100 50  0001 L BNN "Field4"
+F 5 "Unavailable" H 4050 4100 50  0001 L BNN "Field5"
+F 6 "SMD IC MCU 32BIT 512KB FLASH 84MHz" H 4050 4100 50  0001 L BNN "Field6"
+F 7 "ATSAM3X8EA-AU-ND" H 4050 4100 50  0001 L BNN "Field7"
+F 8 "None" H 4050 4100 50  0001 L BNN "Field8"
+	1    4050 4100
+	1    0    0    -1
+$EndComp
+Wire Wire Line
+	5800 1350 6400 1350
+$Comp
+L Connector:USB_OTG J21
+U 1 1 5B6CC522
+P 700 3750
+F 0 "J21" H 755 4217 50  0000 C CNN
+F 1 "USB_OTG" H 755 4126 50  0000 C CNN
+F 2 "Connectors_USB:USB_Micro-B_Molex-105017-0001" H 850 3700 50  0001 C CNN
+F 3 " ~" H 850 3700 50  0001 C CNN
+	1    700  3750
+	1    0    0    -1
+$EndComp
+Wire Wire Line
+	600  4150 700  4150
+Connection ~ 700  4150
+Wire Wire Line
+	1700 5950 1000 5950
+Wire Wire Line
+	1700 5850 1000 5850
+Wire Wire Line
+	1700 5750 1000 5750
+Text HLabel 1000 5750 0    50   Input ~ 0
+TEMP1
+Text HLabel 1000 5850 0    50   Input ~ 0
+TEMP2
+Text HLabel 1000 5950 0    50   Input ~ 0
+TEMP3
+$Comp
+L Connector:Conn_ARM_JTAG_SWD_10 J25
+U 1 1 5B6F5E59
+P 6450 7200
+F 0 "J25" H 6009 7154 50  0000 R CNN
+F 1 "Conn_ARM_JTAG_SWD_10" H 6009 7245 50  0000 R CNN
+F 2 "Connectors_Harwin:Harwin_Gecko-G125-FVX1005L0X_2x05x1.25mm_Straight" H 6500 6650 50  0001 L TNN
+F 3 "http://infocenter.arm.com/help/topic/com.arm.doc.faqs/attached/13634/cortex_debug_connectors.pdf" V 6100 5950 50  0001 C CNN
+	1    6450 7200
+	-1   0    0    1
+$EndComp
 $EndSCHEMATC

Commit message: Added additional PCB layout
Parts:
- C1, C2, C3, C4: value C -> 22p
Connections:
- net labels removed: VDDHMI
Changed lines of the file:
@@
 P 650 2500
 F 0 "C4" V 398 2500 50  0000 C CNN
-F 1 "C" V 489 2500 50  0000 C CNN
+F 1 "22p" V 489 2500 50  0000 C CNN
 F 2 "Capacitors_SMD:C_0805" H 688 2350 50  0001 C CNN
 F 3 "~" H 650 2500 50  0001 C CNN
@@
 P 600 2050
 F 0 "C2" V 348 2050 50  0000 C CNN
-F 1 "C" V 439 2050 50  0000 C CNN
+F 1 "22p" V 439 2050 50  0000 C CNN
 F 2 "Capacitors_SMD:C_0805" H 638 1900 50  0001 C CNN
 F 3 "~" H 600 2050 50  0001 C CNN
@@
 P 600 1650
 F 0 "C1" V 348 1650 50  0000 C CNN
-F 1 "C" V 439 1650 50  0000 C CNN
+F 1 "22p" V 439 1650 50  0000 C CNN
 F 2 "Capacitors_SMD:C_0805" H 638 1500 50  0001 C CNN
 F 3 "~" H 600 1650 50  0001 C CNN
@@
 P 650 2250
 F 0 "C3" V 398 2250 50  0000 C CNN
-F 1 "C" V 489 2250 50  0000 C CNN
+F 1 "22p" V 489 2250 50  0000 C CNN
 F 2 "Capacitors_SMD:C_0805" H 688 2100 50  0001 C CNN
 F 3 "~" H 650 2250 50  0001 C CNN
@@
 $EndComp
 Text Label 9150 2850 0    50   ~ 0
-VDDHMI
+VDDMI
 Text Label 9950 2850 0    50   ~ 0
 VDDANA

Commit message: Added Motor driver revision 1.0
Connections:
- wire segments 130 -> 152
Changed lines of the file:
@@
 L Device:Ferrite_Bead L4
 U 1 1 5B26AB18
-P 5400 850
-F 0 "L4" V 5126 850 50  0000 C CNN
-F 1 "Ferrite_Bead" V 5217 850 50  0000 C CNN
-F 2 "Inductors_SMD:L_0805" V 5330 850 50  0001 C CNN
-F 3 "~" H 5400 850 50  0001 C CNN
-	1    5400 850
+P 5550 850
+F 0 "L4" V 5276 850 50  0000 C CNN
+F 1 "Ferrite_Bead" V 5367 850 50  0000 C CNN
+F 2 "Inductors_SMD:L_0805" V 5480 850 50  0001 C CNN
+F 3 "~" H 5550 850 50  0001 C CNN
+	1    5550 850
 	0    1    1    0
 $EndComp
@@
 	3100 1350 3100 1150
 Wire Wire Line
-	3600 1100 4300 1100
+	3600 1100 3700 1100
 Wire Wire Line
 	4300 1100 4300 1350
@@
 	5750 850  5750 650
 Wire Wire Line
-	5550 850  5750 850
-Wire Wire Line
 	6600 650  6600 1150
-Wire Wire Line
-	6600 1150 4700 1150
 Wire Wire Line
 	4700 1150 4700 1350
@@
 	3600 1100 3600 1350
 Wire Wire Line
-	4900 850  5250 850
-Wire Wire Line
 	6350 650  6600 650
 Wire Wire Line
@@
 	-1   0    0    1
 $EndComp
+Wire Wire Line
+	3700 1350 3700 1100
+Connection ~ 3700 1100
+Wire Wire Line
+	3700 1100 3800 1100
+Wire Wire Line
+	3800 1350 3800 1100
+Connection ~ 3800 1100
+Wire Wire Line
+	3800 1100 3900 1100
+Wire Wire Line
+	3900 1350 3900 1100
+Connection ~ 3900 1100
+Wire Wire Line
+	3900 1100 4000 1100
+Wire Wire Line
+	4000 1350 4000 1100
+Connection ~ 4000 1100
+Wire Wire Line
+	4000 1100 4300 1100
+Wire Wire Line
+	5500 1350 5600 1350
+Wire Wire Line
+	5700 1350 5600 1350
+Connection ~ 5600 1350
+Wire Wire Line
+	5700 1350 5800 1350
+Connection ~ 5700 1350
+Connection ~ 5800 1350
+Wire Wire Line
+	6400 1750 6400 1850
+Connection ~ 6400 1750
+Wire Wire Line
+	6400 1850 6400 1950
+Connection ~ 6400 1850
+Wire Wire Line
+	6400 1950 6400 2050
+Connection ~ 6400 1950
+Connection ~ 6400 2050
+Wire Wire Line
+	4700 1150 6600 1150
+Wire Wire Line
+	5700 850  5750 850
+Wire Wire Line
+	4900 850  5000 850
+Wire Wire Line
+	5300 1350 5300 850
+Connection ~ 5300 850
+Wire Wire Line
+	5300 850  5400 850
+Wire Wire Line
+	5200 1350 5200 850
+Connection ~ 5200 850
+Wire Wire Line
+	5200 850  5300 850
+Wire Wire Line
+	5100 1350 5100 850
+Connection ~ 5100 850
+Wire Wire Line
+	5100 850  5200 850
+Wire Wire Line
+	5000 1350 5000 850
+Connection ~ 5000 850
+Wire Wire Line
+	5000 850  5100 850
 $EndSCHEMATC

Commit message: Added updates to controller hardware
Parts:
- added D2, D3, D6: LED, Diodes_SMD:D_0805, symbol PrinterController-rescue:LED
- added R16, R18, R19, R20: 330R, Resistors_SMD:R_0805, symbol PrinterController-rescue:R
- D1: footprint Capacitors_Tantalum_SMD:CP_Tantalum_Case-B_EIA-3528-21_Hand -> Diodes_SMD:D_0805
Connections:
- wire segments 152 -> 173
Changed lines of the file:
@@
 F 0 "D1" H 5400 7600 50  0000 C CNN
 F 1 "LED" H 5400 7400 50  0000 C CNN
-F 2 "Capacitors_Tantalum_SMD:CP_Tantalum_Case-B_EIA-3528-21_Hand" H 5400 7500 50  0001 C CNN
+F 2 "Diodes_SMD:D_0805" H 5400 7500 50  0001 C CNN
 F 3 "" H 5400 7500 50  0001 C CNN
 	1    5400 7500
@@
 	1    0    0    -1
 $EndComp
-Wire Wire Line
-	5800 1350 6400 1350
 $Comp
 L Connector:USB_OTG J21
@@
 	4000 1100 4300 1100
 Wire Wire Line
-	5500 1350 5600 1350
-Wire Wire Line
-	5700 1350 5600 1350
-Connection ~ 5600 1350
-Wire Wire Line
-	5700 1350 5800 1350
-Connection ~ 5700 1350
-Connection ~ 5800 1350
-Wire Wire Line
-	6400 1750 6400 1850
-Connection ~ 6400 1750
-Wire Wire Line
-	6400 1850 6400 1950
-Connection ~ 6400 1850
-Wire Wire Line
-	6400 1950 6400 2050
-Connection ~ 6400 1950
-Connection ~ 6400 2050
-Wire Wire Line
 	4700 1150 6600 1150
 Wire Wire Line
@@
 Wire Wire Line
 	5000 850  5100 850
+$Comp
+L PrinterController-rescue:LED D2
+U 1 1 5B73BA54
+P 850 4550
+F 0 "D2" H 850 4650 50  0000 C CNN
+F 1 "LED" H 850 4450 50  0000 C CNN
+F 2 "Diodes_SMD:D_0805" H 850 4550 50  0001 C CNN
+F 3 "" H 850 4550 50  0001 C CNN
+	1    850  4550
+	0    -1   -1   0
+$EndComp
+$Comp
+L PrinterController-rescue:R R20
+U 1 1 5B73BA5C
+P 3750 7700
+F 0 "R20" V 3830 7700 50  0000 C CNN
+F 1 "330R" V 3750 7700 50  0000 C CNN
+F 2 "Resistors_SMD:R_0805" V 3680 7700 50  0001 C CNN
+F 3 "" H 3750 7700 50  0001 C CNN
+	1    3750 7700
+	0    1    1    0
+$EndComp
+Wire Wire Line
+	3900 7700 3900 7650
+$Comp
+L PrinterController-rescue:R R16
+U 1 1 5B756055
+P 700 4750
+F 0 "R16" V 780 4750 50  0000 C CNN
+F 1 "330R" V 700 4750 50  0000 C CNN
+F 2 "Resistors_SMD:R_0805" V 630 4750 50  0001 C CNN
+F 3 "" H 700 4750 50  0001 C CNN
+	1    700  4750
+	0    -1   -1   0
+$EndComp
+$Comp
+L PrinterController-rescue:R R18
+U 1 1 5B7562B6
+P 700 4850
+F 0 "R18" V 750 4550 50  0000 C CNN
+F 1 "330R" V 700 4850 50  0000 C CNN
+F 2 "Resistors_SMD:R_0805" V 630 4850 50  0001 C CNN
+F 3 "" H 700 4850 50  0001 C CNN
+	1    700  4850
+	0    -1   -1   0
+$EndComp
+$Comp
+L PrinterController-rescue:R R19
+U 1 1 5B756326
+P 700 4950
+F 0 "R19" V 600 5050 50  0000 C CNN
+F 1 "330R" V 700 4950 50  0000 C CNN
+F 2 "Resistors_SMD:R_0805" V 630 4950 50  0001 C CNN
+F 3 "" H 700 4950 50  0001 C CNN
+	1    700  4950
+	0    -1   -1   0
+$EndComp
+$Comp
+L PrinterController-rescue:LED D3
+U 1 1 5B7565E9
+P 1100 4550
+F 0 "D3" H 1100 4650 50  0000 C CNN
+F 1 "LED" H 1100 4450 50  0000 C CNN
+F 2 "Diodes_SMD:D_0805" H 1100 4550 50  0001 C CNN
+F 3 "" H 1100 4550 50  0001 C CNN
+	1    1100 4550
+	0    -1   -1   0
+$EndComp
+$Comp
+L PrinterController-rescue:LED D6
+U 1 1 5B756665
+P 1350 4550
+F 0 "D6" H 1350 4650 50  0000 C CNN
+F 1 "LED" H 1350 4450 50  0000 C CNN
+F 2 "Diodes_SMD:D_0805" H 1350 4550 50  0001 C CNN
+F 3 "" H 1350 4550 50  0001 C CNN
+	1    1350 4550
+	0    -1   -1   0
+$EndComp
+Connection ~ 6400 2050
+Connection ~ 6400 1950
+Connection ~ 6400 1850
+Connection ~ 6400 1750
+Connection ~ 5800 1350
+Connection ~ 5700 1350
+Connection ~ 5600 1350
+Wire Wire Line
+	5700 1350 5800 1350
+Wire Wire Line
+	5800 1350 6400 1350
+Wire Wire Line
+	6400 1950 6400 2050
+Wire Wire Line
+	6400 1850 6400 1950
+Wire Wire Line
+	6400 1750 6400 1850
+Wire Wire Line
+	5700 1350 5600 1350
+Wire Wire Line
+	5500 1350 5600 1350
+Wire Wire Line
+	1700 3550 1300 3550
+Wire Wire Line
+	1300 3550 1300 4150
+Wire Wire Line
+	1300 4150 850  4150
+Wire Wire Line
+	850  4150 850  4400
+Wire Wire Line
+	1100 4400 1100 4200
+Wire Wire Line
+	1100 4200 1350 4200
+Wire Wire Line
+	1350 4200 1350 3650
+Wire Wire Line
+	1350 3650 1700 3650
+Wire Wire Line
+	1700 3750 1400 3750
+Wire Wire Line
+	1400 3750 1400 4250
+Wire Wire Line
+	1400 4250 1350 4250
+Wire Wire Line
+	1350 4250 1350 4400
+Wire Wire Line
+	850  4700 850  4750
+Wire Wire Line
+	850  4850 1100 4850
+Wire Wire Line
+	1100 4850 1100 4700
+Wire Wire Line
+	1350 4700 1350 4950
+Wire Wire Line
+	1350 4950 850  4950
+$Comp
+L power:GND #PWR0123
+U 1 1 5B78F350
+P 550 5150
+F 0 "#PWR0123" H 550 4900 50  0001 C CNN
+F 1 "GND" H 555 4977 50  0000 C CNN
+F 2 "" H 550 5150 50  0001 C CNN
+F 3 "" H 550 5150 50  0001 C CNN
+	1    550  5150
+	1    0    0    -1
+$EndComp
+Wire Wire Line
+	550  5150 550  4950
+Wire Wire Line
+	550  4950 550  4850
+Connection ~ 550  4950
+Wire Wire Line
+	550  4850 550  4750
+Connection ~ 550  4850
 $EndSCHEMATC

Commit message: Library update for ATSAM
Connections:
- wire segments 173 -> 174
Changed lines of the file:
@@
 	550  4850 550  4750
 Connection ~ 550  4850
+Wire Wire Line
+	1000 5350 1700 5350
 $EndSCHEMATC
